File: HW/Robot/Servo_Current_Limiter/Servo_Current_Limiter.kicad_pcb (KiCad board)
At the start: 2 copper layers, 54 parts, among them J1 1x3 2.54mm male, J10 1x3 2.54mm male, J11 1x1 2.54mm male, J12 1x1 2.54mm male, J13 1x3 2.54mm male, J14 1x1 2.54mm male, J2 Conn_02x05_Odd_Even, J3 1x1 2.54mm male, J4 1x3 2.54mm male, J5 1x1 2.54mm male, J6 1x1 2.54mm male, J7 1x3 2.54mm male, J8 1x1 2.54mm male, J9 1x1 2.54mm male, Q1 IRF4905, Q2 BC548, Q3 IRF4905, Q4 BC548, Q5 IRF4905, Q6 BC548, Q7 IRF4905, Q8 BC548, U1 LM324

Commit message: Something done.
Parts:
- added JP2: 1x2 2.54mm male, Connector_PinHeader_2.54mm:PinHeader_1x02_P2.54mm_Vertical, F.Cu at (58.4, 169.9)
- added JP3: 1x2 2.54mm male, Connector_PinHeader_2.54mm:PinHeader_1x02_P2.54mm_Vertical, F.Cu at (141.8, 332.5)
- added JP4: 1x2 2.54mm male, Connector_PinHeader_2.54mm:PinHeader_1x02_P2.54mm_Vertical, F.Cu at (141.8, 322.1)
- added JP5: 1x2 2.54mm male, Connector_PinHeader_2.54mm:PinHeader_1x02_P2.54mm_Vertical, F.Cu at (129.5, 322.1)
- added R25: 100k, For_Rasterboard:R_Axial_DIN0207_L6.3mm_D2.5mm_P7.62mm_Horizontal, F.Cu at (61.0, 169.9)
- added R26: 10k, For_Rasterboard:R_Axial_DIN0207_L6.3mm_D2.5mm_Pinf_Horizontal, F.Cu at (149.1, 267.4)
- added R27: 10k, For_Rasterboard:R_Axial_DIN0207_L6.3mm_D2.5mm_Pinf_Horizontal, F.Cu at (135.1, 283.3)
- added R28: 10k, For_Rasterboard:R_Axial_DIN0207_L6.3mm_D2.5mm_P7.62mm_Horizontal, F.Cu at (68.6, 172.4)
- added R29: 10k, Resistor_THT:R_Axial_DIN0207_L6.3mm_D2.5mm_P5.08mm_Vertical, F.Cu at (73.7, 177.6)
- added R30: 100k, For_Rasterboard:R_Axial_DIN0207_L6.3mm_D2.5mm_Pinf_Horizontal, F.Cu at (159.9, 267.4)
- added R31: 100k, For_Rasterboard:R_Axial_DIN0207_L6.3mm_D2.5mm_P7.62mm_Horizontal, F.Cu at (109.2, 276.6)
- added R32: 10k, For_Rasterboard:R_Axial_DIN0207_L6.3mm_D2.5mm_Pinf_Horizontal, F.Cu at (190.2, 267.4)
- added R33: 10k, For_Rasterboard:R_Axial_DIN0207_L6.3mm_D2.5mm_Pinf_Horizontal, F.Cu at (176.2, 283.3)
- added R34: 10k, For_Rasterboard:R_Axial_DIN0207_L6.3mm_D2.5mm_P7.62mm_Horizontal, F.Cu at (189.5, 279.3)
- added R35: 10k, Resistor_THT:R_Axial_DIN0207_L6.3mm_D2.5mm_P5.08mm_Vertical, F.Cu at (176.2, 279.3)
- added R36: 100k, For_Rasterboard:R_Axial_DIN0207_L6.3mm_D2.5mm_Pinf_Horizontal, F.Cu at (200.9, 267.4)
- added R37: 100k, For_Rasterboard:R_Axial_DIN0207_L6.3mm_D2.5mm_P7.62mm_Horizontal, F.Cu at (217.3, 243.0)
- added R38: 10k, For_Rasterboard:R_Axial_DIN0207_L6.3mm_D2.5mm_Pinf_Horizontal, F.Cu at (190.2, 243.0)
- added R39: 10k, For_Rasterboard:R_Axial_DIN0207_L6.3mm_D2.5mm_Pinf_Horizontal, F.Cu at (176.2, 258.9)
- added R40: 10k, For_Rasterboard:R_Axial_DIN0207_L6.3mm_D2.5mm_P7.62mm_Horizontal, F.Cu at (189.5, 254.9)
- added R41: 10k, Resistor_THT:R_Axial_DIN0207_L6.3mm_D2.5mm_P5.08mm_Vertical, F.Cu at (176.2, 254.9)
- added R42: 100k, For_Rasterboard:R_Axial_DIN0207_L6.3mm_D2.5mm_Pinf_Horizontal, F.Cu at (200.9, 243.0)
- added R43: 100k, For_Rasterboard:R_Axial_DIN0207_L6.3mm_D2.5mm_P7.62mm_Horizontal, F.Cu at (135.1, 291.9)
- added R44: 10k, For_Rasterboard:R_Axial_DIN0207_L6.3mm_D2.5mm_Pinf_Horizontal, F.Cu at (149.1, 243.0)
- added R45: 10k, For_Rasterboard:R_Axial_DIN0207_L6.3mm_D2.5mm_Pinf_Horizontal, F.Cu at (135.1, 258.9)
- added R46: 10k, For_Rasterboard:R_Axial_DIN0207_L6.3mm_D2.5mm_P7.62mm_Horizontal, F.Cu at (148.4, 254.9)
- added R47: 10k, Resistor_THT:R_Axial_DIN0207_L6.3mm_D2.5mm_P5.08mm_Vertical, F.Cu at (135.1, 254.9)
- added R48: 100k, For_Rasterboard:R_Axial_DIN0207_L6.3mm_D2.5mm_Pinf_Horizontal, F.Cu at (159.9, 243.0)
- added RV5: 1k, Potentiometer_THT:Potentiometer_Piher_PT-10-V10_Vertical, F.Cu at (135.5, 274.0)
- added RV6: 1k, Potentiometer_THT:Potentiometer_Piher_PT-10-V10_Vertical, F.Cu at (176.6, 274.0)
- added RV7: 1k, Potentiometer_THT:Potentiometer_Piher_PT-10-V10_Vertical, F.Cu at (176.6, 249.6)
- added RV8: 1k, Potentiometer_THT:Potentiometer_Piher_PT-10-V10_Vertical, F.Cu at (135.5, 249.6)
- R1, R13, R19, R7: value 220 -> 1k
- R10, R16, R22: footprint For_Rasterboard:R_Axial_DIN0207_L6.3mm_D2.5mm_P7.62mm_Horizontal -> For_Rasterboard:R_Axial_DIN0207_L6.3mm_D2.5mm_P12.70mm_Horizontal
- R11, R17, R23: footprint Resistor_THT:R_Axial_DIN0207_L6.3mm_D2.5mm_P10.16mm_Horizontal -> Resistor_THT:R_Axial_DIN0207_L6.3mm_D2.5mm_P2.54mm_Vertical
- R5: footprint For_Rasterboard:R_Axial_DIN0207_L6.3mm_D2.5mm_P2.54mm_Vertical -> Resistor_THT:R_Axial_DIN0207_L6.3mm_D2.5mm_P2.54mm_Vertical
- RV1, RV2, RV3, RV4: value 250 -> 1k
Routing:
- net /DIS0: track 53.3 -> 58.4 mm

Commit message: Working.
Parts:
- removed J10, J13, J7: 1x3 2.54mm male, Connector_PinHeader_2.54mm:PinHeader_1x03_P2.54mm_Vertical
- removed J11, J12, J14, J6, J8, J9: 1x1 2.54mm male, Connector_PinHeader_2.54mm:PinHeader_1x01_P2.54mm_Vertical
- removed JP3, JP4, JP5: 1x2 2.54mm male, Connector_PinHeader_2.54mm:PinHeader_1x02_P2.54mm_Vertical
- removed Q2, Q4, Q6, Q8: BC548, For_Rasterboard:TO-92_Inline_inf
- removed Q3, Q5, Q7: IRF4905, Package_TO_SOT_THT:TO-220-3_Vertical
- removed R10, R16, R22: 10k, For_Rasterboard:R_Axial_DIN0207_L6.3mm_D2.5mm_P12.70mm_Horizontal
- removed R11, R17, R23: 10k, Resistor_THT:R_Axial_DIN0207_L6.3mm_D2.5mm_P2.54mm_Vertical
- removed R12, R18, R24: 100k, For_Rasterboard:R_Axial_DIN0207_L6.3mm_D2.5mm_P2.54mm_Vertical
- removed R13, R19: 1k, For_Rasterboard:R_Axial_DIN0207_L6.3mm_D2.5mm_Pinf_Horizontal
- removed R14, R20, R8: 0.1, For_Rasterboard:R_Axial_DIN0207_L6.3mm_D2.5mm_P7.62mm_Horizontal
- removed R15, R21, R36, R42, R48, R9: 100k, For_Rasterboard:R_Axial_DIN0207_L6.3mm_D2.5mm_Pinf_Horizontal
- removed R31, R37, R43: 100k, For_Rasterboard:R_Axial_DIN0207_L6.3mm_D2.5mm_P7.62mm_Horizontal
- removed R32, R33, R38, R39, R44, R45: 10k, For_Rasterboard:R_Axial_DIN0207_L6.3mm_D2.5mm_Pinf_Horizontal
- removed R34, R40, R46: 10k, For_Rasterboard:R_Axial_DIN0207_L6.3mm_D2.5mm_P7.62mm_Horizontal
- removed R35, R41, R47: 10k, Resistor_THT:R_Axial_DIN0207_L6.3mm_D2.5mm_P5.08mm_Vertical
- removed RV2, RV3, RV4, RV6, RV7, RV8: 1k, Potentiometer_THT:Potentiometer_Piher_PT-10-V10_Vertical
- R30: value 100k -> 1k
- moved R7 193.1 mm to (95.2, 205.5)
- moved RV5 103.7 mm to (53.4, 210.7)
- moved R26 96.0 mm to (71.8, 210.6)
- moved R27 96.0 mm to (57.8, 226.5)
- moved R30 96.0 mm to (82.5, 210.6)
Connections:
- J3 pad 1: Net-(J3-Pad1) -> /DIS0
- Q1 pad 1: /DIS0 -> /ch0/CTRL
- R25 pad 2: /DIS0 -> /ch0/CTRL
- R7 pad 1: +5V -> /ch0/CTRL
- R7 pad 2: Net-(R7-Pad2) -> GND
- RV1 pad 2: Net-(J3-Pad1) -> /DIS0
- U1 pad 10: Net-(R16-Pad2) -> (no net)
- U1 pad 12: Net-(R22-Pad2) -> (no net)
- U1 pad 13: Net-(R23-Pad1) -> (no net)
- U1 pad 14: /OUT3 -> (no net)
- U1 pad 5: Net-(R10-Pad2) -> /OUT0
- U1 pad 6: Net-(R11-Pad1) -> /DIS0
- U1 pad 7: /OUT1 -> /ch0/CTRL
- U1 pad 8: /OUT2 -> (no net)
- U1 pad 9: Net-(R17-Pad1) -> (no net)
Routing:
- net /ch0/CTRL: track 0.00 -> 94.0 mm, vias 0 -> 3
- net /OUT1: track 63.5 -> 12.7 mm, vias 2 -> 1
- net /DIS0: track 58.4 -> 17.8 mm, vias 3 -> 1
- net Net-(J3-Pad1): track 17.8 -> 0.00 mm, vias 1 -> 0
- net /OUT0: track 68.6 -> 78.7 mm, vias 5 -> 4
- net /ch0/P: track 7.62 -> 12.7 mm
