File: HW/Robot/Servo_Current_Limiter/Servo_Current_Limiter.kicad_sch (KiCad schematic)
At the start: 6 parts, among them J1 1x3 2.54mm male, J2 Conn_02x05_Odd_Even, U1 LM324

Commit message: Working.
Other:
- removed sheet ch1
- removed sheet ch2
- removed sheet ch3
